Commit message: Update vajra.xacro

File: vajra/urdf/vajra.xacro (robot description, xacro)
@@ -8,29 +8,4 @@
         <origin xyz="0.0 0.0 0.010" rpy="0 0 0"/>
     </joint>
-    <joint name="counter_weight_joint" type="fixed">
-        <parent link="base_link"/>
-        <child link="counter_weight_link"/>
-        <origin xyz="0.5 0.0 0.1" rpy="0 0 0"/>
-    </joint>
-    <link name="counter_weight_link">
-        <visual>
-            <origin rpy="0 0 0" xyz="0 0 0"/>
-            <geometry>
-                <box size="0.1 0.1 0.1"/>
-            </geometry>
-        </visual>
-        <inertial>
-            <origin xyz="0 0 0" rpy="0 0 0"/>
-            <mass value="1"/>
-            <inertia ixx="0.00166666666667" ixy="0.0" ixz="0.0" iyy="0.00166666666667" iyz="0.0"
-                     izz="0.00166666666667"/>
-        </inertial>
-        <collision>
-            <origin xyz="0 0 0" rpy="0 0 0"/>
-            <geometry>
-                <box size="0.02 0.02 0.02"/>
-            </geometry>
-        </collision>
-    </link>
     <link name="base_link">
         <visual>
